File: PCB/MotorBoard/MotorBoard.kicad_pcb (KiCad board)
At the start: 2 copper layers, 35 x 35 mm, 16 parts, among them IC1 DRV8874PWPR, J1 Power, J2 Conn_01x06_Pin, J3 Conn_01x06_Pin, J4 Conn_01x03_Pin, J5 Conn_01x04_Pin, J6 Conn_01x04_Pin, U1 ATtiny1617-M

Commit message: Some minor changes
Parts:
- added C6: 1uF, Capacitor_SMD:C_0603_1608Metric, F.Cu at (53.2, 75.8)
- C4: footprint Capacitor_SMD:C_0603_1608Metric -> Capacitor_Tantalum_SMD:CP_EIA-7343-15_Kemet-W
- C5: value 10uF -> 0.1uF; footprint Capacitor_Tantalum_SMD:CP_EIA-7343-40_Kemet-Y -> Capacitor_SMD:C_0603_1608Metric
- moved J6 47.9 mm to (62.5, 91.8), turned to 145 degrees
- moved U1 46.2 mm to (57.9, 77.8)
- moved C4 45.1 mm to (41.0, 86.7), turned to 180 degrees
- moved C3 44.5 mm to (43.5, 90.8), turned to 180 degrees
- moved C2 41.0 mm to (48.2, 90.2), turned to -90 degrees
- moved C1 40.4 mm to (50.0, 90.0), turned to -90 degrees
- moved C5 40.2 mm to (53.2, 74.2)
- moved J3 40.0 mm to (46.2, 66.2)
- moved R1 38.4 mm to (47.0, 78.2), turned to 90 degrees
- moved J5 36.9 mm to (66.8, 83.2), turned to 180 degrees
- moved R2 36.6 mm to (49.0, 78.2), turned to -90 degrees
- moved J4 20.6 mm to (63.8, 70.3), turned to 30 degrees
- moved J1 9.72 mm to (39.6, 79.3), turned to 75 degrees
- moved IC1 1.25 mm to (48.5, 84.4)
Connections:
- C5 pad 1: Net-(U1-VCC) -> +3.3V
- J3 pad 2: +5V -> +3.3V
- J3 pad 3: /CS -> /SS
- J3 pad 4: /CLK -> /SCK
- U1 pad 10: /EncoderB -> /EncoderA
- U1 pad 4: Net-(U1-VCC) -> +3.3V
- U1 pad 7: /EncoderA -> /EncoderB
Routing:
- net +3.3V: track 0.00 -> 85.6 mm, vias 0 -> 1
- net GND: track 0.00 -> 34.7 mm, vias 0 -> 31
- net /ADC2: track 0.00 -> 28.4 mm
- net +12V: track 0.00 -> 23.4 mm, vias 0 -> 2
- net /SCK: track 0.00 -> 20.6 mm
- net /SS: track 0.00 -> 20.2 mm
- net /IPROPI: track 0.00 -> 19.7 mm, vias 0 -> 2
- net /MOSI: track 0.00 -> 16.0 mm
- net /NSLEEP: track 0.00 -> 16.0 mm, vias 0 -> 2
- net /NFAULT: track 0.00 -> 15.4 mm, vias 0 -> 2
- net /EncoderB: track 0.00 -> 14.4 mm
- net /EncoderA: track 0.00 -> 13.9 mm
- net /MotorA: track 0.00 -> 12.6 mm
- net /EN/IN1: track 0.00 -> 12.1 mm, vias 0 -> 2
- net /RESET/UPDI: track 0.00 -> 11.3 mm, vias 0 -> 1
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- added copper zone on B.Cu, net GND
- added copper zone on F.Cu, net GND
