File: PCB/MainBoard/MainBoard.kicad_pcb (KiCad board)
At the start: 2 copper layers, 11 parts, among them IC1 ICM-42670-P, J1 USB_C_Receptacle_USB2.0_14P, J2 Conn_01x06_Pin, J3 Conn_01x06_Pin, J4 Conn_01x06_Pin, J5 Conn_01x06_Pin, U2 ESP32-S3-WROOM-1

Commit message: Added some 3D models to components
Other:
- board outline added: 66 x 44 mm
Changed lines of the file:
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@@
+			)
+		)
+		(model "${KICAD9_3DMODEL_DIR}/RF_Module.3dshapes/ESP32-WROOM-32U.wrl"
+			(offset
+				(xyz 0 0 0)
+			)
+			(scale
+				(xyz 1 1 1)
+			)
+			(rotate
+				(xyz 0 0 0)
 			)
 		)
@@
 			)
 		)
+		(model "${KICAD9_3DMODEL_DIR}/Connector_USB.3dshapes/USB_C_Receptacle_GCT_USB4105-xx-A_16P_TopMnt_Horizontal.wrl"
+			(offset
+				(xyz 0 0 0)
+			)
+			(scale
+				(xyz 1 1 1)
+			)
+			(rotate
+				(xyz 0 0 0)
+			)
+		)
 	)
 	(footprint "Connector_JST:JST_PH_B6B-PH-K_1x06_P2.00mm_Vertical"
@@
 		)
 	)
+	(gr_rect
+		(start 69 65)
+		(end 135 109)
+		(stroke
+			(width 0.05)
+			(type default)
+		)
+		(fill no)
+		(layer "Edge.Cuts")
+	)
 	(embedded_fonts no)
